File: kicad/iaq_device/iaq_device.kicad_pcb (KiCad board)
At the start: 2 copper layers, 70.1 x 43.2 mm, 19 parts, among them J1 External Pins, SW1 B3S-1000, SW2 CO2 CAL, U1 WeMos_D1_mini, U2 PMS7003, U3 SSD1306, U4 BME280, U5 MH-Z19, U6 SGP30, U7 TSL2561T

Commit message: Initial commit of c3 board
Parts:
- removed ?: , 
- removed U1: WeMos_D1_mini, Nikolay Library:WEMOS_D1_surface
- added U8: ~, footprints:ESP32-C3 SUPERMINI, F.Cu at (99.7, 96.1)
- JP1: footprint Jumper:SolderJumper-3_P1.3mm_Open_RoundedPad1.0x1.5mm_NumberLabels -> Jumper:SolderJumper-3_P1.3mm_Open_RoundedPad1.0x1.5mm
- U3: footprint Nikolay Library:SSD1306 -> footprints:SSD1306_I2C_0.96in
- moved SW2 47.9 mm to (172.7, 110.4)
- moved U4 23.3 mm to (176.0, 90.3), turned to 180 degrees
- moved U6 19.9 mm to (169.2, 83.6), turned to 0 degrees
- moved U3 8.50 mm to (166.6, 102.9), turned to 180 degrees
- moved C2 8.00 mm to (116.5, 114.2), turned to 180 degrees
- moved C4 8.00 mm to (135.3, 114.2), turned to 180 degrees
- moved C3 8.00 mm to (125.6, 114.2), turned to 180 degrees
- moved JP1 5.08 mm to (107.2, 101.3), turned to 0 degrees
- moved SW1 2.28 mm to (143.2, 110.3)
- moved U5 0.63 mm to (162.9, 114.3)
- moved J1 0.57 mm to (137.5, 92.6)
Connections:
- D3 pad 4: (no net) -> unconnected-(D3-DO-Pad4)
- U2 pad 5: (no net) -> unconnected-(U2-Reset-Pad5)
- U2 pad 6: (no net) -> unconnected-(U2-Pad6)
- U2 pad 7: (no net) -> unconnected-(U2-RX-Pad7)
- U2 pad 8: (no net) -> unconnected-(U2-Pad8)
- U5 pad 1: (no net) -> unconnected-(U5-Vout-Pad1)
- U5 pad 4: (no net) -> unconnected-(U5-SR-Pad4)
- U5 pad 8: (no net) -> unconnected-(U5-AOT-Pad8)
- U5 pad 9: (no net) -> unconnected-(U5-PWM-Pad9)
- U7 pad 5: (no net) -> unconnected-(U7-INT-Pad5)
Routing:
- net SDA: track 76.3 -> 158.9 mm, vias 2 -> 0
- net SCL: track 94.1 -> 170.2 mm, vias 4 -> 0
- net +5V: track 148.3 -> 196.5 mm, vias 3 -> 2
- net D8: track 40.7 -> 0.00 mm, vias 2 -> 0
- net +3V3: track 124.9 -> 152.2 mm, vias 2 -> 3
- net GND: track 31.8 -> 7.74 mm, vias 19 -> 34
- net Net-(U8-0): track 50.2 -> 73.9 mm
- net D3: track 23.2 -> 0.00 mm, vias 2 -> 0
- net PMS_SET: track 33.7 -> 11.8 mm, vias 3 -> 0
- net Net-(U5-CAL): track 44.6 -> 23.2 mm
- net PMS_RX: track 30.9 -> 15.9 mm, vias 2 -> 0
- net MH_TX: track 63.7 -> 50.4 mm, vias 3 -> 0
- net A0: track 24.8 -> 37.1 mm, vias 2 -> 0
- net LED_D: track 10.2 -> 17.0 mm, vias 2 -> 0
- net MH_RX: track 56.1 -> 50.8 mm, vias 3 -> 0
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Other:
- board size 70.1 x 43.2 mm -> 78.2 x 43.2 mm
- net class Default removed
- board text added: "ESP32-C3 Air Quality Board rev.1.0"
- board text added: "https://github.com/noisymime/iaq_board-c3"
- board text removed: "Wemos D1 Mini Air Quality Board rev.1.1"
- board text removed: "https://github.com/nkitanov/iaq_board"

Commit message: v2.0 of the C3 PCB files
Parts:
- removed J1: External Pins, Connector_PinSocket_2.54mm:PinSocket_1x08_P2.54mm_Vertical_SMD_Pin1Left
- SW1: value B3S-1000 -> SEL; footprint Nikolay Library:SW_SPST_B3S-1000 -> Button_Switch_SMD:SW_SPST_TL3305B
- SW2: footprint Button_Switch_SMD:SW_SPST_B3U-1000P -> Button_Switch_SMD:SW_SPST_TL3342
- U6: moved to F.Cu
- moved U6 22.5 mm to (150.6, 96.3), turned to 180 degrees
- moved SW1 14.4 mm to (133.5, 99.7), turned to 0 degrees
- moved JP1 9.06 mm to (103.3, 109.5), turned to -90 degrees
- moved U8 6.34 mm to (101.5, 102.2)
- moved U5 6.11 mm to (167.4, 110.1)
- moved U2 0.76 mm to (124.5, 96.0), turned to 0 degrees
- moved SW2 0.29 mm to (173.0, 110.5), turned to -90 degrees
Connections:
- SW1 pad 1: Net-(U8-0) -> Net-(U8-7)
- U8 pad 4: unconnected-(U8-6-Pad4) -> D6
- U8 pad 6: unconnected-(U8-7-Pad6) -> Net-(U8-7)
- U8 pad 9: Net-(U8-0) -> unconnected-(U8-3-Pad9)
Routing:
- net Net-(U8-0): track 73.9 -> 0.00 mm, vias 2 -> 0
- net A0: track 37.1 -> 0.00 mm
- net PMS_SET: track 11.8 -> 43.8 mm
- net Net-(U8-7): track 0.00 -> 31.8 mm
- net SCL: track 170.2 -> 138.8 mm
- net PMS_RX: track 15.9 -> 41.7 mm
- net +5V: track 196.5 -> 221.8 mm, vias 2 -> 1
- net Net-(JP1-C): track 18.5 -> 3.00 mm
- net SDA: track 158.9 -> 147.1 mm, vias 0 -> 2
- net +3V3: track 152.2 -> 158.9 mm, vias 3 -> 2
- net LED_D: track 17.0 -> 11.0 mm
- net GND: track 7.74 -> 3.62 mm, vias 34 -> 42
- net Net-(U5-CAL): track 23.2 -> 21.3 mm
- net MH_TX: track 50.4 -> 51.1 mm
Other:
- rule solder_mask_min_width: 0.25 -> 0.2
- board text added: "ESP32-C3 Air Quality Board rev.2.0"
- board text removed: "1"
- board text removed: "3.3V"
- board text removed: "5V"
- board text removed: "A0"
- board text removed: "D3"
- board text removed: "D8"
- board text removed: "ESP32-C3 Air Quality Board rev.1.0"
- board text removed: "GND"
- board text removed: "SCL"
