File: kicad/iaq_device/iaq_device.kicad_sch (KiCad schematic)
At the start: 18 parts, among them J1 External Pins, SW1 B3S-1000, SW2 CO2 CAL, U2 PMS7003, U3 SSD1306, U4 BME280, U5 MH-Z19, U6 SGP30, U7 TSL2561T

Commit message: v2.0 of the C3 PCB files
Parts:
- removed J1: External Pins, Connector_PinSocket_2.54mm:PinSocket_1x08_P2.54mm_Vertical_SMD_Pin1Left, symbol Connector_Generic:Conn_01x08
- SW1: value B3S-1000 -> SEL; footprint Nikolay Library:SW_SPST_B3S-1000 -> Button_Switch_SMD:SW_SPST_TL3305B; eshop https://uk.farnell.com/omron/b3s-1000/switch-spno-0-05a-24v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 -> https://www.digikey.com.au/en/products/detail/e-switch/TL33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
- SW2: footprint Button_Switch_SMD:SW_SPST_B3U-1000P -> Button_Switch_SMD:SW_SPST_TL3342; eshop https://bg.farnell.com/omron/b3u-1000p/switch-spst-no-0-05a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 -> https://www.digikey.com.au/en/products/detail/e-switch/TL33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
Connections:
- net at SW1.1: now also U8.6 (7); no longer U8.9 (3)
- net D6: now reaches U8.4 (6)
- no-connect marks 10 -> 8
Other:
- moved on the sheet: SW1, U8

Commit message: Updated design files
Parts:
- C1, C2, C3, C4: eshop https://bg.farnell.com/wurth-elektronik/885012207016/cap-0-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 -> https://www.digikey.com.au/en/products/detail/w%C3%BCrth-el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
Changed lines of the file:
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@@
       (effects (font (size 1.27 1.27)) hide)
     )
-    (property "eshop" "https://bg.farnell.com/wurth-elektronik/885012207016/cap-0-1-f-10v-10-x7r-0805/dp/2534051?st=smd%20capacitors" (at 158.75 77.47 0)
+    (property "eshop" "https://www.digikey.com.au/en/products/detail/w%C3%BCrth-elektronik/885012207016/5453881" (at 158.75 77.47 0)
       (effects (font (size 1.27 1.27)) hide)
     )
@@
       (effects (font (size 1.27 1.27)) hide)
     )
-    (property "eshop" "https://bg.farnell.com/wurth-elektronik/885012207016/cap-0-1-f-10v-10-x7r-0805/dp/2534051?st=smd%20capacitors" (at 82.55 123.19 0)
+    (property "eshop" "https://www.digikey.com.au/en/products/detail/w%C3%BCrth-elektronik/885012207016/5453881" (at 82.55 123.19 0)
       (effects (font (size 1.27 1.27)) hide)
     )
@@
       (effects (font (size 1.27 1.27)) hide)
     )
-    (property "eshop" "https://bg.farnell.com/wurth-elektronik/885012207016/cap-0-1-f-10v-10-x7r-0805/dp/2534051?st=smd%20capacitors" (at 104.14 123.19 0)
+    (property "eshop" "https://www.digikey.com.au/en/products/detail/w%C3%BCrth-elektronik/885012207016/5453881" (at 104.14 123.19 0)
       (effects (font (size 1.27 1.27)) hide)
     )
@@
       (effects (font (size 1.27 1.27)) hide)
     )
-    (property "eshop" "https://bg.farnell.com/wurth-elektronik/885012207016/cap-0-1-f-10v-10-x7r-0805/dp/2534051?st=smd%20capacitors" (at 125.73 123.19 0)
-      (effects (font (size 1.27 1.27)) hide)
-    )
+    (property "eshop" "https://www.digikey.com.au/en/products/detail/w%C3%BCrth-elektronik/885012207016/5453881" (at 125.73 123.19 0)
+      (effects (font (size 1.27 1.27)) hide)
+    )
